Commit message: update kinect model

File: bluerov2_hdt/urdf/sensors/kinect.urdf.xacro (robot description, xacro)
@@ -55,5 +55,5 @@
 				<origin xyz="0.0 0.0 0.0" rpy="0.0 0.0 0"/>
 				<geometry>
-					<mesh filename="package://sensors_description/meshes/sensors/kinect.dae" scale="1 1 1" />
+					<mesh filename="package://bluerov2_hdt/meshes/sensors/kinect.dae" scale="1 1 1" />
 				</geometry>
 				<material name="gray">
@@ -64,5 +64,5 @@
 				<origin xyz="0.0 0.0 0.0" rpy="0.0 0.0 0.0"/>
 				<geometry>
-					<mesh filename="package://sensors_description/meshes/sensors/kinect.dae" scale="1 1 1" />
+					<mesh filename="package://bluerov2_hdt/meshes/sensors/kinect.dae" scale="1 1 1" />
 				</geometry>
 			</collision>

Commit message: update kinect urdf model

File: bluerov2_hdt/urdf/sensors/kinect.urdf.xacro (robot description, xacro)
@@ -55,5 +55,5 @@
 				<origin xyz="0.0 0.0 0.0" rpy="0.0 0.0 0"/>
 				<geometry>
-					<mesh filename="package://bluerov2_hdt/meshes/sensors/kinect.dae" scale="1 1 1" />
+					<mesh filename="package://bluerov2_hdt/meshes/kinect.dae" scale="1 1 1" />
 				</geometry>
 				<material name="gray">
@@ -64,5 +64,5 @@
 				<origin xyz="0.0 0.0 0.0" rpy="0.0 0.0 0.0"/>
 				<geometry>
-					<mesh filename="package://bluerov2_hdt/meshes/sensors/kinect.dae" scale="1 1 1" />
+					<mesh filename="package://bluerov2_hdt/meshes/kinect.dae" scale="1 1 1" />
 				</geometry>
 			</collision>

File: bluerov2_hdt/urdf/sensors/stereo_snippets.xacro (robot description, xacro)
@@ -41,5 +41,5 @@
       <visual>
         <geometry>
-          <mesh filename="file://$(find c)/meshes/duo3d.dae"/>
+          <mesh filename="file://$(find bluerov2_hdt)/meshes/duo3d.dae"/>
         </geometry>
       </visual>
