Commit message: update stereo camera

File: bluerov2_hdt/robots/bluerov2_hdt.xacro (robot description, xacro)
@@ -13,4 +13,11 @@
 -->
 <robot name="bluerov2" xmlns:xacro="http://wiki.ros.org/xacro" >
+  <!-- Loading file with sensor macros -->
+  <!-- <xacro:include filename="$(find uuv_sensor_ros_plugins)/urdf/sensor_snippets.xacro"/> -->
+  <xacro:include filename="$(find bluerov2_hdt)/urdf/sensors/stereo_snippets.xacro"/>
+  <!-- <xacro:include filename="$(find bluerov2_hdt)/urdf/sensors/kinect.urdf.xacro"/> -->
+  <!-- <xacro:include filename="$(find sensors_description)/urdfs/sensors/kinect.urdf.xacro"/> -->
+  <xacro:include filename="$(find bluerov2_hdt)/urdf/sensors/kinect.urdf.xacro"/>
+  <!-- <xacro:include filename="$(find sensors_description)/urdfs/common.xacro"/> -->
   <!-- <xacro:arm name="update_rate" default="10"/> -->
   <xacro:arg name="debug" default="0"/>
@@ -99,3 +106,14 @@
     </sensor>
   </gazebo>
+  <xacro:kinect_camera name="$(arg namespace)/kinect_camera" parent="$(arg namespace)/base_link">
+    <origin xyz="0.25 0 -0.1" rpy="0 0 0"/>
+  </xacro:kinect_camera>
+   <!-- Mount a stereo camera -->
+  <xacro:duo3d_camera namespace="$(arg namespace)" parent_link="$(arg namespace)/base_link">
+    <origin xyz="0.25 0 0." rpy="0 0 0"/>
+  </xacro:duo3d_camera>
+  <!-- Mount a camera -->
+  <!-- <xacro:default_camera namespace="${namespace}" parent_link="${namespace}/base_link" suffix="front">
+    <origin xyz="0 0 0.2" rpy="0 0 0"/>
+  </xacro:default_camera> -->
 </robot>

Commit message: update duo3d urdf model

File: bluerov2_hdt/robots/bluerov2_hdt.xacro (robot description, xacro)
@@ -14,10 +14,6 @@
 <robot name="bluerov2" xmlns:xacro="http://wiki.ros.org/xacro" >
   <!-- Loading file with sensor macros -->
-  <!-- <xacro:include filename="$(find uuv_sensor_ros_plugins)/urdf/sensor_snippets.xacro"/> -->
-  <xacro:include filename="$(find bluerov2_hdt)/urdf/sensors/stereo_snippets.xacro"/>
-  <!-- <xacro:include filename="$(find bluerov2_hdt)/urdf/sensors/kinect.urdf.xacro"/> -->
-  <!-- <xacro:include filename="$(find sensors_description)/urdfs/sensors/kinect.urdf.xacro"/> -->
+  <xacro:include filename="$(find bluerov2_hdt)/urdf/sensors/duo3d_snippets.xacro"/>
   <xacro:include filename="$(find bluerov2_hdt)/urdf/sensors/kinect.urdf.xacro"/>
-  <!-- <xacro:include filename="$(find sensors_description)/urdfs/common.xacro"/> -->
   <!-- <xacro:arm name="update_rate" default="10"/> -->
   <xacro:arg name="debug" default="0"/>
@@ -110,7 +106,7 @@
   </xacro:kinect_camera>
    <!-- Mount a stereo camera -->
-  <xacro:duo3d_camera namespace="$(arg namespace)" parent_link="$(arg namespace)/base_link">
+  <xacro:duo3d_stereo_camera namespace="$(arg namespace)" parent_link="$(arg namespace)/base_link">
     <origin xyz="0.25 0 0." rpy="0 0 0"/>
-  </xacro:duo3d_camera>
+  </xacro:duo3d_stereo_camera>
   <!-- Mount a camera -->
   <!-- <xacro:default_camera namespace="${namespace}" parent_link="${namespace}/base_link" suffix="front">

File: bluerov2_hdt/urdf/sensors/duo3d_snippets.xacro (robot description, xacro)
@@ -13,10 +13,10 @@
 -->
 <robot xmlns:xacro="http://www.ros.org/wiki/xacro">
-  <xacro:property name="k1l" value="-0.0"/>
+  <xacro:property name="k1l" value="0.0"/>
   <xacro:property name="k2l" value="0.0"/>
   <xacro:property name="p1l" value="0.0"/>
   <xacro:property name="p2l" value="0.0"/>
   <xacro:property name="k3l" value="0.0"/>
-  <xacro:property name="k1r" value="-0.0"/>
+  <xacro:property name="k1r" value="0.0"/>
   <xacro:property name="k2r" value="0.0"/>
   <xacro:property name="p1r" value="0.0"/>
@@ -33,5 +33,5 @@
     </collision>
   </xacro:macro>
-  <xacro:macro name="duo3d_camera" params="namespace parent_link *origin">
+  <xacro:macro name="duo3d_stereo_camera" params="namespace parent_link *origin">
     <link name="${namespace}/duo3d_left_link">
       <inertial>
@@ -41,5 +41,5 @@
       <visual>
         <geometry>
-          <mesh filename="file://$(find bluerov2_hdt)/meshes/duo3d.dae"/>
+          <mesh filename="package://bluerov2_hdt/meshes/duo3d.dae"/>
         </geometry>
       </visual>
@@ -67,9 +67,9 @@
         </clip>
         <distortion>
-          <k1>${k1l}</k1>
-          <k2>${k2l}</k2>
-          <k3>${k3l}</k3>
-          <p1>${p1l}</p1>
-          <p2>${p2l}</p2>
+          <k1>0</k1>
+          <k2>0</k2>
+          <k3>0</k3>
+          <p1>0</p1>
+          <p2>0</p2>
           <center>0.5 0.5</center>
         </distortion>
@@ -83,9 +83,9 @@
         <frameName>${namespace}/duo3d_left_link</frameName>
         <hackBaseline>0.07</hackBaseline>
-        <distortionK1>${k1l}</distortionK1>
-        <distortionK2>${k2l}</distortionK2>
-        <distortionK3>${k3l}</distortionK3>
-        <distortionT1>${p1l}</distortionT1>
-        <distortionT2>${p2l}</distortionT2>
+        <distortionK1>0</distortionK1>
+        <distortionK2>0</distortionK2>
+        <distortionK3>0</distortionK3>
+        <distortionT1>0</distortionT1>
+        <distortionT2>0</distortionT2>
       </plugin>
       <always_on>1</always_on>
@@ -122,9 +122,9 @@
         </clip>
         <distortion>
-          <k1>${k1l}</k1>
-          <k2>${k2l}</k2>
-          <k3>${k3l}</k3>
-          <p1>${p1l}</p1>
-          <p2>${p2l}</p2>
+          <k1>0</k1>
+          <k2>0</k2>
+          <k3>0</k3>
+          <p1>0</p1>
+          <p2>0</p2>
           <center>0.5 0.5</center>
         </distortion>
@@ -138,9 +138,9 @@
         <frameName>${namespace}/duo3d_right_link</frameName>
         <hackBaseline>0.07</hackBaseline>
-        <distortionK1>${k1l}</distortionK1>
-        <distortionK2>${k2l}</distortionK2>
-        <distortionK3>${k3l}</distortionK3>
-        <distortionT1>${p1l}</distortionT1>
-        <distortionT2>${p2l}</distortionT2>
+        <distortionK1>0</distortionK1>
+        <distortionK2>0</distortionK2>
+        <distortionK3>0</distortionK3>
+        <distortionT1>0</distortionT1>
+        <distortionT2>0</distortionT2>
       </plugin>
       <always_on>1</always_on>
